File: PowerStation/PowerStation.kicad_pcb (KiCad board)
At the start: 2 copper layers, 25 parts, among them J1 Salidas, J14 ReguladorExterno, J15 ReguladorExterno, J2 12VA, J3 12VB, J4 12VC, J5 12VD, J6 12VE, J7 3V3, J8 5V, J9 Conn_01x05_Pin, K1 Relay_SPDT, K6 Relay_SPDT, U1 ACS712xLCTR-20A, U2 ACS712xLCTR-20A, U4 LM4040DBZ-4.1

Commit message: avanxe en placa
Parts:
- added C1: 1nF, Capacitor_SMD:C_0402_1005Metric, F.Cu at (111.8, 85.3)
- added C2: C, Capacitor_SMD:C_0402_1005Metric, F.Cu at (111.8, 87.3)
- added C3: 100nF, Capacitor_SMD:C_0402_1005Metric, F.Cu at (111.8, 89.2)
- added C4: 100nF, Capacitor_SMD:C_0402_1005Metric, F.Cu at (111.8, 91.2)
- added C5: 10 uF, Capacitor_SMD:C_0402_1005Metric, F.Cu at (116.7, 87.3)
- added C6: 0.1 uF, Capacitor_SMD:C_0402_1005Metric, F.Cu at (116.7, 89.3)
- added J10: GND, Connector_JST:JST_ZE_B10B-ZESK-D_1x10_P1.50mm_Vertical, F.Cu at (79.3, 115.0)
- added J11: GND, Connector_JST:JST_ZE_B10B-ZESK-D_1x10_P1.50mm_Vertical, F.Cu at (54.0, 130.9)
- added J12: GND, Connector_JST:JST_ZE_B10B-ZESK-D_1x10_P1.50mm_Vertical, F.Cu at (65.0, 135.7)
- added J13: GND, Connector_JST:JST_ZE_B10B-ZESK-D_1x10_P1.50mm_Vertical, F.Cu at (22.2, 117.2)
- added K2: Relay_SPDT, Relay_THT:Relay_SPDT_Finder_36.11, F.Cu at (176.4, 51.9)
- added K3: Relay_SPDT, Relay_THT:Relay_SPDT_Finder_36.11, F.Cu at (176.4, 69.0)
- added K4: Relay_SPDT, Relay_THT:Relay_SPDT_Finder_36.11, F.Cu at (176.4, 86.0)
- added K5: Relay_SPDT, Relay_THT:Relay_SPDT_Finder_36.11, F.Cu at (176.4, 103.0)
- added R1: 330, Resistor_SMD:R_0402_1005Metric, F.Cu at (116.7, 93.2)
- added R2: 330, Resistor_SMD:R_0402_1005Metric, F.Cu at (116.7, 95.2)
- added R3: 1M ohm, Resistor_SMD:R_0402_1005Metric, F.Cu at (108.9, 85.3)
- added R4: 100K ohm, Resistor_SMD:R_0402_1005Metric, F.Cu at (108.9, 87.3)
- added R5: 1M ohm, Resistor_SMD:R_0402_1005Metric, F.Cu at (108.9, 89.3)
- added R6: 100K ohm, Resistor_SMD:R_0402_1005Metric, F.Cu at (108.9, 91.3)
- added R7: 909 ohm, Resistor_SMD:R_0402_1005Metric, F.Cu at (116.7, 85.3)
- added SW1: SW_Push_Dual, Connector:FanPinHeader_1x04_P2.54mm_Vertical, F.Cu at (222.5, 75.1)
- added SW2: SW_Push_Dual, Connector:FanPinHeader_1x04_P2.54mm_Vertical, F.Cu at (222.5, 89.0)
- J9: value Conn_01x05_Pin -> control
- moved J1 140.0 mm to (221.9, 114.4), turned to 90 degrees
- moved J8 89.3 mm to (80.0, 137.6), turned to 90 degrees
- moved J9 81.4 mm to (28.9, 83.8), turned to 90 degrees
- moved J5 80.4 mm to (52.1, 84.0), turned to -90 degrees
- moved J7 80.3 mm to (68.9, 111.7), turned to 90 degrees
- moved K6 77.2 mm to (176.4, 137.2)
- moved K1 77.1 mm to (176.4, 120.1)
- moved J14 74.5 mm to (202.5, 68.8)
- moved J15 73.8 mm to (204.4, 88.6)
- moved U2 72.0 mm to (205.5, 99.0)
- moved U1 70.0 mm to (204.4, 78.9)
- moved J6 69.8 mm to (52.1, 99.7), turned to -90 degrees
- moved J3 68.8 mm to (52.1, 64.8), turned to -90 degrees
- moved J4 68.8 mm to (52.1, 74.4), turned to -90 degrees
- moved D8 61.9 mm to (167.1, 133.9)
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
Commit message: correccion de esquermatico y avanze en placa
Parts:
- removed SW1, SW2: SW_Push_Dual, Connector:FanPinHeader_1x04_P2.54mm_Vertical
- removed U4: LM4040DBZ-4.1, Package_TO_SOT_SMD:SOT-23
- added C7: 10nF, Capacitor_SMD:C_0402_1005Metric, F.Cu at (126.3, 38.8)
- added C8: 10nF, Capacitor_SMD:C_0402_1005Metric, F.Cu at (143.8, 135.2)
- added D10: 1N4007, Diode_SMD:D_SMA, F.Cu at (132.7, 112.0)
- added D9: 1N4007, Diode_SMD:D_SMA, F.Cu at (135.2, 51.8)
- added J16: Salida 1, Connector:JWT_A3963_1x02_P3.96mm_Vertical, F.Cu at (165.1, 49.7)
- added K7: Relay_SPDT, Relay_THT:Relay_SPDT_Finder_36.11, F.Cu at (139.5, 51.3)
- added K8: Relay_SPDT, Relay_THT:Relay_SPDT_Finder_36.11, F.Cu at (138.3, 112.4)
- added U3: ACS712xLCTR-20A, Package_SO:SOIC-8_3.9x4.9mm_P1.27mm, F.Cu at (138.1, 134.0)
- C1: value 1nF -> 0.1 uF
- C2: value C -> 10 uF
- C3: value 100nF -> 1nF
- C5: value 10 uF -> 100nF
- C6: value 0.1 uF -> 1nf
- D1, D2: value LED -> 1N4007; footprint LED_SMD:LED_0805_2012Metric -> Diode_SMD:D_SMA
- D3, D4, D5, D6: value D -> 1N4007; footprint Diode_SMD:D_01005_0402Metric -> Diode_SMD:D_SMA
- D7, D8: value D -> LED; footprint Diode_SMD:D_01005_0402Metric -> LED_SMD:LED_0805_2012Metric
- J1: value Salidas -> 12VA; footprint Connector_JST:JST_NV_B04P-NV_1x04_P5.00mm_Vertical -> Connector_JST:JST_ZE_B05B-ZESK-D_1x05_P1.50mm_Vertical
- J10: value GND -> 5V; footprint Connector_JST:JST_ZE_B10B-ZESK-D_1x10_P1.50mm_Vertical -> Connector_JST:JST_ZE_B09B-ZESK-1D_1x09_P1.50mm_Vertical
- J11: value GND -> 12VE; footprint Connector_JST:JST_ZE_B10B-ZESK-D_1x10_P1.50mm_Vertical -> Connector_JST:JST_ZE_B05B-ZESK-D_1x05_P1.50mm_Vertical
- J12: value GND -> 3V3
- J13: value GND -> Salida 2; footprint Connector_JST:JST_ZE_B10B-ZESK-D_1x10_P1.50mm_Vertical -> Connector:JWT_A3963_1x02_P3.96mm_Vertical
- J2: value 12VA -> control
- J4: value 12VC -> GND; footprint Connector_JST:JST_ZE_B03B-ZESK-D_1x03_P1.50mm_Vertical -> Connector_JST:JST_ZE_B10B-ZESK-D_1x10_P1.50mm_Vertical
- J5: value 12VD -> GND; footprint Connector_JST:JST_ZE_B07B-ZESK-D_1x07_P1.50mm_Vertical -> Connector_JST:JST_ZE_B10B-ZESK-D_1x10_P1.50mm_Vertical
- J6: value 12VE -> 12VC; footprint Connector_JST:JST_ZE_B05B-ZESK-D_1x05_P1.50mm_Vertical -> Connector_JST:JST_ZE_B03B-ZESK-D_1x03_P1.50mm_Vertical
- J7: value 3V3 -> 12VD; footprint Connector_JST:JST_ZE_B10B-ZESK-D_1x10_P1.50mm_Vertical -> Connector_JST:JST_ZE_B07B-ZESK-D_1x07_P1.50mm_Vertical
- J8: value 5V -> GND; footprint Connector_JST:JST_ZE_B09B-ZESK-1D_1x09_P1.50mm_Vertical -> Connector_JST:JST_ZE_B10B-ZESK-D_1x10_P1.50mm_Vertical
- J9: value control -> GND; footprint Connector_JST:JST_ZE_B05B-ZESK-D_1x05_P1.50mm_Vertical -> Connector_JST:JST_ZE_B10B-ZESK-D_1x10_P1.50mm_Vertical
- R1: value 330 -> 909 ohm
- R2: value 330 -> 1M ohm
- R3, R5: value 1M ohm -> 100K ohm
- R4: value 100K ohm -> 1M ohm
- R6: value 100K ohm -> 330
- R7: value 909 ohm -> 330
- U1: value ACS712xLCTR-20A -> LM4040DBZ-4.1; footprint Package_SO:SOIC-8_3.9x4.9mm_P1.27mm -> Package_TO_SOT_SMD:SOT-23
- moved U1 178.9 mm to (32.8, 28.4), turned to 90 degrees
- moved J1 160.4 mm to (64.6, 83.2), turned to 0 degrees
- moved J13 144.0 mm to (166.2, 111.9), turned to -90 degrees
- moved J15 133.8 mm to (90.4, 158.6)
- moved K1 125.5 mm to (83.5, 35.8)
- moved J14 124.4 mm to (88.2, 19.9)
- moved R1 107.8 mm to (29.7, 29.7), turned to 180 degrees
- moved D6 105.1 mm to (74.7, 131.3), turned to 90 degrees
- moved C2 101.7 mm to (29.7, 27.2), turned to 180 degrees
- moved C1 99.9 mm to (29.7, 28.4), turned to 180 degrees
- moved D4 98.0 mm to (74.7, 98.3), turned to 90 degrees
- moved U2 95.6 mm to (127.7, 43.4), turned to 90 degrees
- moved K4 93.7 mm to (83.5, 98.0)
- moved K5 93.7 mm to (83.5, 114.8)
- moved D5 93.5 mm to (74.7, 115.9), turned to 90 degrees
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Connections:
- A1 pad 14: unconnected-(A1-D11-Pad14) -> /control/digitalPin10
- A1 pad 15: unconnected-(A1-D12-Pad15) -> /control/digitalPin11
- A1 pad 18: Net-(A1-AREF) -> /control/AREF
- C1 pad 1: Net-(U1-FILTER) -> /control/5V
- C2 pad 1: Net-(U2-FILTER) -> /control/5V
- C3 pad 1: /control/analogIN1 -> Net-(U2-FILTER)
- C4 pad 1: /control/analogIN3 -> /control/analogIN1
- C5 pad 1: /control/5V -> /control/analogIN3
- C6 pad 1: /control/5V -> Net-(U3-FILTER)
- D1 pad 1: GND -> /control de salidas/relay1S1
- D1 pad 2: Net-(D1-A) -> GND
- D2 pad 1: GND -> /control de salidas/relay2S1
- D2 pad 2: Net-(D2-A) -> GND
- D3 pad 1: /control de salidas/relay2S1 -> /control de salidas/relay3S1
- D4 pad 1: /control de salidas/relay1S1 -> /control de salidas/relay1S2
- D5 pad 1: /control de salidas/relay3S1 -> /control de salidas/relay2S2
- D6 pad 1: /control de salidas/relay1S2 -> /control de salidas/relay3S2
- D7 pad 1: /control de salidas/relay2S2 -> GND
- D7 pad 2: GND -> Net-(D7-A)
- D8 pad 1: /control de salidas/relay3S2 -> GND
- D8 pad 2: GND -> Net-(D8-A)
- J1 pad 1: Net-(J1-Pin_1) -> /control de salidas/12VA
- J1 pad 2: Net-(J1-Pin_2) -> /control de salidas/12VA
- J1 pad 3: GND -> /control de salidas/12VA
- J1 pad 4: GND -> /control de salidas/12VA
- J10 pad 1: GND -> /control de salidas/5V
- J10 pad 2: GND -> /control de salidas/5V
- J10 pad 3: GND -> /control de salidas/5V
- J10 pad 4: GND -> /control de salidas/5V
- J10 pad 5: GND -> /control de salidas/5V
- J10 pad 6: GND -> /control de salidas/5V
- J10 pad 7: GND -> /control de salidas/5V
- J10 pad 8: GND -> /control de salidas/5V
- J10 pad 9: GND -> /control de salidas/5V
- J11 pad 1: GND -> /entrada de fuente/12VE
- J11 pad 2: GND -> /entrada de fuente/12VE
- J11 pad 3: GND -> /entrada de fuente/12VE
- J11 pad 4: GND -> /entrada de fuente/12VE
- J11 pad 5: GND -> /entrada de fuente/12VE
- J12 pad 1: GND -> /control de salidas/3V3
- J12 pad 10: GND -> unconnected-(J12-Pin_10-Pad10)
- J12 pad 2: GND -> /control de salidas/3V3
- J12 pad 3: GND -> /control de salidas/3V3
- J12 pad 4: GND -> /control de salidas/3V3
- J12 pad 5: GND -> /control de salidas/3V3
- J12 pad 6: GND -> /control de salidas/3V3
- J12 pad 7: GND -> /control de salidas/3V3
- J12 pad 8: GND -> /control de salidas/3V3
- J12 pad 9: GND -> /control de salidas/3V3
- J13 pad 2: GND -> Net-(J13-Pin_2)
- J2 pad 1: /control de salidas/12VA -> /entrada de fuente/-12V
- J2 pad 2: /control de salidas/12VA -> /control/5V
- J2 pad 3: /control de salidas/12VA -> /control/digitalPin7
- J2 pad 4: /control de salidas/12VA -> /control/digitalPin8
- J2 pad 5: /control de salidas/12VA -> /control/digitalPin9
- J4 pad 1: /control de salidas/12VC -> GND
- J4 pad 2: /control de salidas/12VC -> GND
- J4 pad 3: /control de salidas/12VC -> GND
- J5 pad 1: /control de salidas/12VD -> GND
- J5 pad 2: /control de salidas/12VD -> GND
- J5 pad 3: /control de salidas/12VD -> GND
- J5 pad 4: /control de salidas/12VD -> GND
- J5 pad 5: /control de salidas/12VD -> GND
- J5 pad 6: /control de salidas/12VD -> GND
- J5 pad 7: /control de salidas/12VD -> GND
- J6 pad 1: /entrada de fuente/12VE -> /control de salidas/12VC
- J6 pad 2: /entrada de fuente/12VE -> /control de salidas/12VC
- J6 pad 3: /entrada de fuente/12VE -> /control de salidas/12VC
- J7 pad 1: /control de salidas/3V3 -> /control de salidas/12VD
- J7 pad 2: /control de salidas/3V3 -> /control de salidas/12VD
- J7 pad 3: /control de salidas/3V3 -> /control de salidas/12VD
- J7 pad 4: /control de salidas/3V3 -> /control de salidas/12VD
- J7 pad 5: /control de salidas/3V3 -> /control de salidas/12VD
- J7 pad 6: /control de salidas/3V3 -> /control de salidas/12VD
- J7 pad 7: /control de salidas/3V3 -> /control de salidas/12VD
- J8 pad 1: /control de salidas/5V -> GND
- J8 pad 2: /control de salidas/5V -> GND
- J8 pad 3: /control de salidas/5V -> GND
- J8 pad 4: /control de salidas/5V -> GND
- J8 pad 5: /control de salidas/5V -> GND
- J8 pad 6: /control de salidas/5V -> GND
- J8 pad 7: /control de salidas/5V -> GND
- J8 pad 8: /control de salidas/5V -> GND
- J8 pad 9: /control de salidas/5V -> GND
- J9 pad 1: /entrada de fuente/-12V -> GND
- J9 pad 2: /control/5V -> GND
- J9 pad 3: /control/digitalPin7 -> GND
- J9 pad 4: /control/digitalPin8 -> GND
- J9 pad 5: /control/digitalPin9 -> GND
- K1 pad 11: /control de salidas/Salida1 -> Net-(K1-Pad11)
- K1 pad 12: Net-(K1-Pad12) -> /control de salidas/5V
- K1 pad 14: /control de salidas/12VA -> /control de salidas/Reguladr de voltaje 1/SalidaRegulada2
- K1 pad A1: /control de salidas/relay3S1 -> /control de salidas/relay1S1
- K2 pad 11: Net-(K1-Pad12) -> Net-(K2-Pad11)
- K2 pad 12: Net-(K2-Pad12) -> Net-(K1-Pad11)
- K3 pad 11: Net-(K2-Pad12) -> /control de salidas/Salida1
- K3 pad 12: /control de salidas/5V -> Net-(K2-Pad11)
- K3 pad 14: /control de salidas/Reguladr de voltaje 1/SalidaRegulada2 -> /control de salidas/12VA
- K3 pad A1: /control de salidas/relay1S1 -> /control de salidas/relay3S1
- R1 pad 1: Net-(R1-Pad1) -> /control/5V
- R1 pad 2: Net-(D1-A) -> /control/AREF
- R2 pad 1: Net-(R2-Pad1) -> /medicion de salidas/Entrada1
- R2 pad 2: Net-(D2-A) -> /control/analogIN1
- R3 pad 1: /medicion de salidas/Entrada1 -> /control/analogIN1
- R3 pad 2: /control/analogIN1 -> GND
- R4 pad 1: /control/analogIN1 -> /medicion de salidas/Entrada2
- R4 pad 2: GND -> /control/analogIN3
- R5 pad 1: /medicion de salidas/Entrada2 -> /control/analogIN3
- R5 pad 2: /control/analogIN3 -> GND
- R6 pad 1: /control/analogIN3 -> /control/digitalPin10
- R6 pad 2: GND -> Net-(D7-A)
- R7 pad 1: /control/5V -> /control/digitalPin11
- R7 pad 2: Net-(A1-AREF) -> Net-(D8-A)
- U1 pad 1: /medicion de salidas/Entrada1 -> /control/AREF
- U1 pad 2: /medicion de salidas/Entrada1 -> GND
- U1 pad 3: /medicion de salidas/Salida1 -> (no net)
- U2 pad 1: /medicion de salidas/Entrada2 -> /medicion de salidas/Entrada1
- U2 pad 2: /medicion de salidas/Entrada2 -> /medicion de salidas/Entrada1
- U2 pad 3: /medicion de salidas/Salida2 -> /medicion de salidas/Salida1
- U2 pad 4: /medicion de salidas/Salida2 -> /medicion de salidas/Salida1
- U2 pad 7: /control/analogIN4 -> /control/analogIN2
Routing:
- net /control de salidas/3V3: track 0.00 -> 144.9 mm, vias 0 -> 1
- net /control de salidas/relay3S2: track 0.00 -> 141.8 mm
- net /control de salidas/relay2S2: track 0.00 -> 135.1 mm
- net /control de salidas/relay1S2: track 0.00 -> 115.9 mm
- net /control/5V: track 0.00 -> 73.7 mm
- net /control de salidas/Reguladr de voltaje 2/SalidaRegulada2: track 0.00 -> 61.8 mm
- net /control de salidas/5V: track 0.00 -> 58.6 mm
- net /control/digitalPin8: track 0.00 -> 43.1 mm
- net /control/digitalPin9: track 0.00 -> 43.0 mm
- net /control/digitalPin7: track 0.00 -> 37.4 mm
- net /control de salidas/12VB: track 0.00 -> 36.6 mm
- net /control de salidas/12VD: track 0.00 -> 29.2 mm
- net /control de salidas/Reguladr de voltaje 1/SalidaRegulada2: track 0.00 -> 24.3 mm
- net GND: track 0.00 -> 19.5 mm, vias 0 -> 9
- net Net-(K5-Pad11): track 0.00 -> 18.7 mm
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- added copper zone on F.Cu, net /control de salidas/12VA
- added copper zone on B.Cu, net GND
