File: PowerStation/controlDeSalidas.kicad_sch (KiCad schematic)
At the start: 0 parts

Commit message: terminando diagrama
Parts:
- added D3, D4, D5, D6, D7, D8: D, Diode_SMD:D_01005_0402Metric, symbol Device:D
- added K1, K6: Relay_SPDT, Relay_THT:Relay_SPDT_Finder_36.11, symbol Relay:Relay_SPDT
- added K2, K3, K4, K5: Relay_SPDT, symbol Relay:Relay_SPDT
Connections:
- new net: K1.12, K2.11
- new net: K5.11, K6.12
- new net: K4.11, K5.12
- new net: K2.12, K3.11
- new net 12VA: K1.14
- new net 12VB: K6.14
- new net 3V3: K2.14, K5.14
- new net 5V: K3.12, K4.12
- new net GND: D3.2 (A), D4.2 (A), D5.2 (A), D6.2 (A), D7.2 (A), D8.2 (A), K1.A2, K2.A2, K3.A2, K4.A2, K5.A2, K6.A2
- new net Reguladr de voltaje 1/SalidaRegulada: K3.14
- new net Reguladr de voltaje 2/SalidaRegulada: K4.14
- new net Salida1: K1.11
- new net Salida2: K6.11
- new net relay1S1: D4.1 (K), K3.A1
- new net relay1S2: D6.1 (K), K4.A1
- new net relay2S1: D3.1 (K), K2.A1
- new net relay2S2: D7.1 (K), K5.A1
- new net relay3S1: D5.1 (K), K1.A1
- new net relay3S2: D8.1 (K), K6.A1
Other:
- added sheet Reguladr de voltaje 1 (regulador.kicad_sch)
- added sheet Reguladr de voltaje 2 (regulador.kicad_sch)
- note added: "|---------------------------------------------------------| | Nombre | color |cantidad de cablees| amperaje | |---------------------------------------------------------| | 12VA | amarillo | 5 cables | 18 A | | 12VB | blanco | 3 cables | 18 A | | 12VC | azul blanco | 3 cables | 18 A | | 12VD | amarillo blanco| 7 cables | 18 A | | 12VE | azul amarillo | 5 cables | 18 A | | -12v | AZUL | 1 cable | 0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"

Commit message: avanxe en placa
Parts:
- K2, K3, K4, K5: footprint (none) -> Relay_THT:Relay_SPDT_Finder_36.11
Connections:
- net Reguladr de voltaje 1/SalidaRegulada renamed Reguladr de voltaje 1/SalidaRegulada2
- net Reguladr de voltaje 2/SalidaRegulada renamed Reguladr de voltaje 2/SalidaRegulada2
Other:
- sheet Reguladr de voltaje 1 ports: added SalidaRegulada2; removed SalidaRegulada
- sheet Reguladr de voltaje 2 ports: added SalidaRegulada2; removed SalidaRegulada
- moved on the sheet: D6, D7, D8, K3, K4, K5, K6

Commit message: correccion de esquermatico y avanze en placa
Parts:
- removed D3, D4, D5, D6, D7, D8: D, Diode_SMD:D_01005_0402Metric, symbol Device:D
- added D1, D2, D3, D4, D5, D6: 1N4007, Diode_SMD:D_SMA, symbol PCM_Diode_AKL:1N4007
- renumbered K3 to K1, K1 to K3
Connections:
- net GND: now also D1.2 (A), D2.2 (A), D3.2 (A), D4.2 (A), D5.2 (A), D6.2 (A)
- net relay1S1: now also D1.1 (K)
- net relay1S2: now also D4.1 (K)
- net relay2S1: now also D2.1 (K)
- net relay2S2: now also D5.1 (K)
- net relay3S1: now also D3.1 (K)
- net relay3S2: now also D6.1 (K)
