File: PowerStation/medicionDeSalidas.kicad_sch (KiCad schematic)
At the start: 0 parts

Commit message: terminando diagrama
Parts:
- added C1: 1nF, symbol Device:C
- added C2: C, symbol Device:C
- added C3, C4: 100nF, symbol Device:C
- added R3, R5: 1M ohm, symbol Device:R
- added R4, R6: 100K ohm, symbol Device:R
- added U1, U2: ACS712xLCTR-20A, Package_SO:SOIC-8_3.9x4.9mm_P1.27mm, symbol Sensor_Current:ACS712xLCTR-20A
Connections:
- new net: C1.1, U1.6 (FILTER)
- new net: C2.1, U2.6 (FILTER)
- new net 5V: U1.8 (VCC), U2.8 (VCC)
- new net Entrada1: R3.1, U1.1 (IP+), U1.2 (IP+)
- new net Entrada2: R5.1, U2.1 (IP+), U2.2 (IP+)
- new net GND: C1.2, C2.2, C3.2, C4.2, R4.2, R6.2, U1.5 (GND), U2.5 (GND)
- new net Salida1: U1.3 (IP-), U1.4 (IP-)
- new net Salida2: U2.3 (IP-), U2.4 (IP-)
- new net medCS1: U1.7 (VIOUT)
- new net medCS2: U2.7 (VIOUT)
- new net medVS1: C3.1, R3.2, R4.1
- new net medVS2: C4.1, R5.2, R6.1

Commit message: avanxe en placa
Parts:
- C1, C2, C3, C4: footprint (none) -> Capacitor_SMD:C_0402_1005Metric
- R3, R4, R5, R6: footprint (none) -> Resistor_SMD:R_0402_1005Metric
Changed lines of the file:
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@@
       (effects (font (size 1.27 1.27)) (justify left))
     )
-    (property "Footprint" "" (at 106.172 102.87 90)
+    (property "Footprint" "Resistor_SMD:R_0402_1005Metric" (at 106.172 102.87 90)
       (effects (font (size 1.27 1.27)) hide)
     )
@@
       (effects (font (size 1.27 1.27)) (justify left))
     )
-    (property "Footprint" "" (at 122.8852 87.63 0)
+    (property "Footprint" "Capacitor_SMD:C_0402_1005Metric" (at 122.8852 87.63 0)
       (effects (font (size 1.27 1.27)) hide)
     )
@@
       (effects (font (size 1.27 1.27)) (justify left))
     )
-    (property "Footprint" "" (at 191.4652 83.82 0)
+    (property "Footprint" "Capacitor_SMD:C_0402_1005Metric" (at 191.4652 83.82 0)
       (effects (font (size 1.27 1.27)) hide)
     )
@@
       (effects (font (size 1.27 1.27)) (justify left))
     )
-    (property "Footprint" "" (at 104.902 74.93 90)
+    (property "Footprint" "Resistor_SMD:R_0402_1005Metric" (at 104.902 74.93 90)
       (effects (font (size 1.27 1.27)) hide)
     )
@@
       (effects (font (size 1.27 1.27)) (justify left))
     )
-    (property "Footprint" "" (at 104.902 85.09 90)
+    (property "Footprint" "Resistor_SMD:R_0402_1005Metric" (at 104.902 85.09 90)
       (effects (font (size 1.27 1.27)) hide)
     )
@@
       (effects (font (size 1.27 1.27)) (justify left))
     )
-    (property "Footprint" "" (at 106.172 113.03 90)
+    (property "Footprint" "Resistor_SMD:R_0402_1005Metric" (at 106.172 113.03 90)
       (effects (font (size 1.27 1.27)) hide)
     )
@@
       (effects (font (size 1.27 1.27)) (justify left))
     )
-    (property "Footprint" "" (at 122.8852 115.57 0)
+    (property "Footprint" "Capacitor_SMD:C_0402_1005Metric" (at 122.8852 115.57 0)
       (effects (font (size 1.27 1.27)) hide)
     )
@@
       (effects (font (size 1.27 1.27)) (justify left))
     )
-    (property "Footprint" "" (at 191.4652 127 0)
-      (effects (font (size 1.27 1.27)) hide)
-    )
+    (property "Footprint" "Capacitor_SMD:C_0402_1005Metric" (at 191.4652 127 0)
+      (effects (font (size 1.27 1.27)) hide)
+    )

Commit message: correccion de esquermatico y avanze en placa
Parts:
- added C7, C8: 10nF, Capacitor_SMD:C_0402_1005Metric, symbol Device:C
- C6: renamed from C2; value C -> 1nf
- renumbered C1 to C3, C3 to C4, C4 to C5, R3 to R2, R4 to R3, R5 to R4, R6 to R5, U1 to U2, U2 to U3
Connections:
- net 5V: now also C7.1, C8.1
- net GND: now also C7.2, C8.2
