File: PowerStation/salidas.kicad_sch (KiCad schematic)
At the start: 0 parts

Commit message: terminando diagrama
Parts:
- added D1, D2: LED, LED_SMD:LED_0805_2012Metric, symbol Device:LED
- added J1: Salidas, Connector_JST:JST_NV_B04P-NV_1x04_P5.00mm_Vertical, symbol Connector:Conn_01x04_Socket
- added R1, R2: R, symbol Device:R
- added SW1, SW2: SW_Push_Dual, symbol Switch:SW_Push_Dual
Connections:
- new net: D2.2 (A), R2.2
- new net: R1.1, SW1.4
- new net: D1.2 (A), R1.2
- new net: J1.1 (Pin_1), SW1.2
- new net: J1.2 (Pin_2), SW2.2
- new net: R2.1, SW2.4
- new net 5V: SW1.3, SW2.3
- new net GND: D1.1 (K), D2.1 (K), J1.3 (Pin_3), J1.4 (Pin_4)
- new net Salida1: SW1.1
- new net Salida2: SW2.1

Commit message: avanxe en placa
Parts:
- R1, R2: value R -> 330; footprint (none) -> Resistor_SMD:R_0402_1005Metric
- SW1, SW2: footprint (none) -> Connector:FanPinHeader_1x04_P2.54mm_Vertical
Changed lines of the file:
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@@
       (effects (font (size 1.27 1.27)))
     )
-    (property "Value" "R" (at 114.3 71.12 90)
+    (property "Value" "330" (at 114.3 71.12 90)
       (effects (font (size 1.27 1.27)))
     )
-    (property "Footprint" "" (at 114.3 76.708 90)
+    (property "Footprint" "Resistor_SMD:R_0402_1005Metric" (at 114.3 76.708 90)
       (effects (font (size 1.27 1.27)) hide)
     )
@@
       (effects (font (size 1.27 1.27)))
     )
-    (property "Footprint" "" (at 105.41 64.77 0)
+    (property "Footprint" "Connector:FanPinHeader_1x04_P2.54mm_Vertical" (at 105.41 64.77 0)
       (effects (font (size 1.27 1.27)) hide)
     )
@@
       (effects (font (size 1.27 1.27)))
     )
-    (property "Value" "R" (at 114.3 93.98 90)
+    (property "Value" "330" (at 114.3 93.98 90)
       (effects (font (size 1.27 1.27)))
     )
-    (property "Footprint" "" (at 114.3 99.568 90)
+    (property "Footprint" "Resistor_SMD:R_0402_1005Metric" (at 114.3 99.568 90)
       (effects (font (size 1.27 1.27)) hide)
     )
@@
       (effects (font (size 1.27 1.27)))
     )
-    (property "Footprint" "" (at 105.41 87.63 0)
+    (property "Footprint" "Connector:FanPinHeader_1x04_P2.54mm_Vertical" (at 105.41 87.63 0)
       (effects (font (size 1.27 1.27)) hide)
     )

Commit message: correccion de esquermatico y avanze en placa
Parts:
- removed D2: LED, LED_SMD:LED_0805_2012Metric, symbol Device:LED
- removed J1: Salidas, Connector_JST:JST_NV_B04P-NV_1x04_P5.00mm_Vertical, symbol Connector:Conn_01x04_Socket
- removed R2: 330, Resistor_SMD:R_0402_1005Metric, symbol Device:R
- removed SW1, SW2: SW_Push_Dual, Connector:FanPinHeader_1x04_P2.54mm_Vertical, symbol Switch:SW_Push_Dual
- added D10, D9: 1N4007, Diode_SMD:D_SMA, symbol PCM_Diode_AKL:1N4007
- added D8: LED, LED_SMD:LED_0805_2012Metric, symbol Device:LED
- added J13: Salida 2, Connector:JWT_A3963_1x02_P3.96mm_Vertical, symbol Connector:Conn_01x02_Pin
- added J16: Salida 1, Connector:JWT_A3963_1x02_P3.96mm_Vertical, symbol Connector:Conn_01x02_Pin
- added K7, K8: Relay_SPDT, Relay_THT:Relay_SPDT_Finder_36.11, symbol Relay:Relay_SPDT
- added R7: 330, Resistor_SMD:R_0402_1005Metric, symbol Device:R
- renumbered D1 to D7, R1 to R6
Connections:
- net GND: now also D10.2 (A), D8.1 (K), D9.2 (A), J13.1 (Pin_1), J16.1 (Pin_1), K7.A1, K8.A1
- net Salida1: now also K7.11
- net Salida2: now also K8.11
- net ActSalida1: now reaches R6.1
- net ActSalida1: now also D9.1 (K), K7.A2
- new net: J13.2 (Pin_2), K8.14
- new net: D8.2 (A), R7.2
- new net: J16.2 (Pin_2), K7.14
- new net ActSalida2: D10.1 (K), K8.A2, R7.1
Other:
- moved on the sheet: D7, R6
